Commit message: Added Teleop

File: mecanumbot_description/urdf/mecanumbot.urdf (robot description, URDF)
Before this commit: robot mecanumbot, 6 links, 5 joints
Links:
- link fl_wheel_link: geometry collision sphere radius=${wheel_radius}; visual mesh filename=$(find mecanumbot_description)/meshes/fl_wheel_link.STL scale=1 1 1
- link fr_wheel_link: geometry collision sphere radius=${wheel_radius}; visual mesh filename=$(find mecanumbot_description)/meshes/fr_wheel_link.STL scale=1 1 1
- link rl_wheel_link: geometry collision sphere radius=${wheel_radius}; visual mesh filename=$(find mecanumbot_description)/meshes/rl_wheel_link.STL scale=1 1 1
- link rr_wheel_link: geometry collision sphere radius=${wheel_radius}; visual mesh filename=$(find mecanumbot_description)/meshes/rr_wheel_link.STL scale=1 1 1
Joints:
- joint fl_wheel_joint: axis -1 0 0 -> (none)
- joint fr_wheel_joint: origin xyz=-0.19 0.23 ${wheel_offset_z} rpy=0 0 0 -> xyz=-0.19 0.23 ${wheel_offset_z} rpy=0 0 ${-M_PI/2}
- joint rl_wheel_joint: origin xyz=0.19 -0.23 ${wheel_offset_z} rpy=0 0 0 -> xyz=0.19 -0.23 ${wheel_offset_z} rpy=0 0 ${-M_PI/2}
- joint rr_wheel_joint: origin xyz=0.19 0.23 ${wheel_offset_z} rpy=0 0 0 -> xyz=0.19 0.23 ${wheel_offset_z} rpy=0 0 ${-M_PI/2}

Commit message: ok

File: mecanumbot_description/urdf/mecanumbot.urdf (robot description, URDF)
Before this commit: robot mecanumbot, 6 links, 5 joints
Links:
- added link laser_frame; collision cylinder length=0.04 radius=0.05; visual cylinder length=0.04 radius=0.05
- link fl_wheel_link: geometry collision sphere radius=${wheel_radius}; visual sphere radius=${wheel_radius}
- link fr_wheel_link: geometry collision sphere radius=${wheel_radius}; visual sphere radius=${wheel_radius}
- link rl_wheel_link: geometry collision sphere radius=${wheel_radius}; visual sphere radius=${wheel_radius}
- link rr_wheel_link: geometry collision sphere radius=${wheel_radius}; visual sphere radius=${wheel_radius}
Joints:
- added joint laser_joint: type fixed, parent base_link, child laser_frame, origin xyz=-0.2 0 0.2 rpy=0 0 0
